File: pcb/pic-scr.sch (KiCad schematic (older format))
At the start: 53 parts, among them CN1 USART, J1 Conn_01x02_Male, J2 -5V, J3 0V, J4 MCLR, K1 RELAY, P1 10K, P2 10K, Q1 BTA41-600B, Q2 BC548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

Commit message: Updated shematic and PCB
Parts:
- removed C6: 10nF/250V, Capacitor_THT:C_Rect_L10.0mm_W4.0mm_P7.50mm_MKS4, symbol Device:C
- removed R12: 360R, Resistor_THT:R_Axial_DIN0309_L9.0mm_D3.2mm_P5.08mm_Vertical, symbol Device:R
- added F1: 10A, symbol Device:Fuse
- P1, P2: value 10K -> 25K
- R1: value 220R/2W -> 120Ω/2W
- R10: value 33R -> 33Ω
- R13, R16, R17, R5: value 470R -> 470Ω
- R15: value 3M/0.25W -> 1M/0.25W
- R2: value 27R-33R -> 27Ω-33Ω
- R6: value 150/2W -> 150Ω/2W
Connections:
- wire segments 161 -> 154
Other:
- note added: "7mA Leak!"
- note added: "<-- 4mA"
- note removed: "0.7mA leak"
